File: hermes.kicad_pcb (KiCad board)
At the start: 2 copper layers, 84.2 x 41.1 mm, 24 parts, among them J1 USB_C_Receptacle_USB2.0_16P, P1 USB_C_Plug_USB2.0, U1 XL1509-5.0, U2 MPU-6500, U3 DM-OLED096-636, U4 XL1509-3.3, U5 ESP32-S3

Commit message: old update, now working on new board
Parts:
- added U7: ESP32-S3-WROOM-1, RF_Module:ESP32-S3-WROOM-1, F.Cu at (217.7, 117.3)
- moved P1 5.04 mm to (124.5, 106.0)
- turned R3 to -90 degrees
- renumbered 12VBattery1 to VCC1
Connections:
- U2 pad 23: unconnected-(U2-SCL/SCLK-Pad23) -> SCL
- U5 pad 20: unconnected-(U5-VDD3P3_RTC-Pad20) -> 3V3
- U5 pad 29: unconnected-(U5-VDD_SPI-Pad29) -> 3V3
- U5 pad 46: unconnected-(U5-VDD3P3_CPU-Pad46) -> 3V3
- U5 pad 55: Net-(U5-VDDA-Pad55) -> 3V3
- U5 pad 56: Net-(U5-VDDA-Pad55) -> 3V3
Routing:
- net Net-(U7-GND-Pad1): track 0.00 -> 21.7 mm
- net SCL: track 31.8 -> 43.6 mm, vias 1 -> 4
- net 3V3: track 71.5 -> 81.2 mm
- net GND: track 170.5 -> 177.4 mm
- net Net-(P1-CC): track 4.08 -> 0.12 mm
- net SDA: track 41.1 -> 44.3 mm
Other:
- outline, holes or cut-outs redrawn
