File: hermes.kicad_sch (KiCad schematic)
At the start: 22 parts, among them J1 USB_C_Receptacle_USB2.0_16P, P1 USB_C_Plug_USB2.0, U1 XL1509-5.0, U2 MPU-6500, U3 DM-OLED096-636, U4 XL1509-3.3, U5 ESP32-S3

Commit message: old update, now working on new board
Parts:
- removed R3: 5.1K, Resistor_SMD:R_0201_0603Metric, symbol Device:R
- removed U5: ESP32-S3, Package_DFN_QFN:QFN-56-1EP_7x7mm_P0.4mm_EP4x4mm, symbol MCU_Espressif:ESP32-S3
- added C4: C_US, Capacitor_SMD:C_Elec_3x5.4, symbol Device:C_US
- added U7: ESP32-S3-WROOM-1, RF_Module:ESP32-S3-WROOM-1, symbol RF_Module:ESP32-S3-WROOM-1
Connections:
- net GND: now also U7.1 (GND), U7.40 (GND), U7.41 (GND)
- net SCL: now also U2.23 (SCL/SCLK)
- net USB_D+: now also U7.14 (USB_D+)
- net USB_D-: now also U7.13 (USB_D-)
- no-connect marks 13 -> 2
Other:
- moved on the sheet: R1, R2
